Commit message: commented out joint state publisher in nuturtle description, updated joint names for fake turtle odom, now transforming correctly

File: nuturtle_description/urdf/turtlebot3_burger.urdf.xacro (robot description, xacro)
@@ -39,5 +39,5 @@
     <parent link="base_link"/>
     <child link="wheel_left_link"/>
-    <origin xyz="0.0 ${wheel_base} 0.023" rpy="-1.57 0 0"/>
+    <origin xyz="0.0 ${0.5*wheel_base} 0.023" rpy="-1.57 0 0"/>
     <axis xyz="0 0 1"/>
   </joint>
@@ -67,5 +67,5 @@
     <parent link="base_link"/>
     <child link="wheel_right_link"/>
-    <origin xyz="0.0 -${wheel_base} 0.023" rpy="-1.57 0 0"/>
+    <origin xyz="0.0 -${0.5*wheel_base} 0.023" rpy="-1.57 0 0"/>
     <axis xyz="0 0 1"/>
   </joint>
